Commit message: ㅁㅁ

File: 200_html/urdf/vehicle/vehicle_01.urdf (robot description, URDF)
Before this commit: robot vehicle_4wd, 12 links, 11 joints
Links:
- removed link gear_fl
- removed link gear_fr
- removed link gear_rl
- removed link gear_rr
Joints:
- removed joint joint_gear_fl
- removed joint joint_gear_fr
- removed joint joint_gear_rl
- removed joint joint_gear_rr
- joint joint_fl: mimic joint=joint_gear_fl multiplier=1.0 offset=0.0 -> (none)
- joint joint_fr: mimic joint=joint_gear_fr multiplier=1.0 offset=0.0 -> (none)
- joint joint_rl: mimic joint=joint_gear_rl multiplier=1.0 offset=0.0 -> (none)
- joint joint_rr: mimic joint=joint_gear_rr multiplier=1.0 offset=0.0 -> (none)
