Commit message: **

File: 200_html/urdf/vehicle/vehicle.urdf (robot description, URDF)
Before this commit: robot realistic_vehicle, 5 links, 4 joints
Links:
- added link car_frame, mass 40.0; collision box size=1.02 0.62 0.24; visual box size=0.08 0.56 0.08
- link base_link: mass 38 -> 0.001; geometry 
- link wheel_fl: mass None -> 1.8; geometry collision cylinder length=0.10 radius=0.16; visual cylinder length=0.10 radius=0.16
- link wheel_fr: mass None -> 1.8; geometry collision cylinder length=0.10 radius=0.16; visual cylinder length=0.10 radius=0.16
- link wheel_rl: mass None -> 1.8; geometry collision cylinder length=0.10 radius=0.16; visual cylinder length=0.10 radius=0.16
- link wheel_rr: mass None -> 1.8; geometry collision cylinder length=0.10 radius=0.16; visual cylinder length=0.10 radius=0.16
Joints:
- added joint base_to_car_frame: type fixed, parent base_link, child car_frame, origin xyz=0 0 0 rpy=0 0 0
- joint joint_fl: origin xyz=0.34 0.41 0 rpy=0 0 0 -> xyz=0.33 0.40 0 rpy=0 0 0; parent base_link -> car_frame
- joint joint_fr: origin xyz=0.34 -0.41 0 rpy=0 0 0 -> xyz=0.33 -0.40 0 rpy=0 0 0; parent base_link -> car_frame
- joint joint_rl: origin xyz=-0.34 0.41 0 rpy=0 0 0 -> xyz=-0.33 0.40 0 rpy=0 0 0; parent base_link -> car_frame
- joint joint_rr: origin xyz=-0.34 -0.41 0 rpy=0 0 0 -> xyz=-0.33 -0.40 0 rpy=0 0 0; parent base_link -> car_frame

Commit message: **

File: 200_html/urdf/vehicle/vehicle.urdf (robot description, URDF)
Before this commit: robot vehicle_4wd, 6 links, 5 joints
Links:
- link car_frame: geometry collision box size=1.02 0.62 0.24; visual box size=0.10 0.03 0.004

Commit message: **

File: 200_html/urdf/vehicle/vehicle.urdf (robot description, URDF)
Before this commit: robot vehicle_4wd, 6 links, 5 joints
Links:
- link car_frame: geometry collision box size=1.02 0.62 0.24; visual box size=0.010 0.09 0.035
Joints:
- joint joint_fl: origin xyz=0.33 0.40 0 rpy=0 0 0 -> xyz=0.33 0.40 0.06 rpy=0 0 0
- joint joint_fr: origin xyz=0.33 -0.40 0 rpy=0 0 0 -> xyz=0.33 -0.40 0.06 rpy=0 0 0
- joint joint_rl: origin xyz=-0.33 0.40 0 rpy=0 0 0 -> xyz=-0.33 0.40 0.06 rpy=0 0 0
- joint joint_rr: origin xyz=-0.33 -0.40 0 rpy=0 0 0 -> xyz=-0.33 -0.40 0.06 rpy=0 0 0

Commit message: **

File: 200_html/urdf/vehicle/vehicle.urdf (robot description, URDF)
Before this commit: robot vehicle_4wd, 6 links, 5 joints
Joints:
- joint base_to_car_frame: origin xyz=0 0 0 rpy=0 0 0 -> xyz=0 0 0.10 rpy=0 0 0

Commit message: **

File: 200_html/urdf/vehicle/vehicle.urdf (robot description, URDF)
Before this commit: robot vehicle_4wd, 6 links, 5 joints
Joints:
- joint base_to_car_frame: origin xyz=0 0 0.10 rpy=0 0 0 -> xyz=0 0 0.10 rpy=0 0 1.5707963

Commit message: **

File: 200_html/urdf/vehicle/vehicle.urdf (robot description, URDF)
Before this commit: robot vehicle_4wd, 6 links, 5 joints
Links:
- link car_frame: geometry collision box size=1.02 0.62 0.24; visual box size=0.010 0.09 0.035

Commit message: **

File: 200_html/urdf/vehicle/vehicle.urdf (robot description, URDF)
Before this commit: robot vehicle_4wd, 6 links, 5 joints
Links:
- link wheel_fl: geometry collision cylinder length=0.10 radius=0.16; visual cylinder length=0.030 radius=0.16
- link wheel_fr: geometry collision cylinder length=0.10 radius=0.16; visual cylinder length=0.030 radius=0.16
- link wheel_rl: geometry collision cylinder length=0.10 radius=0.16; visual cylinder length=0.030 radius=0.16
- link wheel_rr: geometry collision cylinder length=0.10 radius=0.16; visual cylinder length=0.030 radius=0.16

Commit message: **

File: 200_html/urdf/vehicle/vehicle.urdf (robot description, URDF)
Before this commit: robot vehicle_4wd, 6 links, 5 joints
Links:
- link wheel_fl: geometry collision cylinder length=0.10 radius=0.16; visual cylinder length=0.08 radius=0.09
- link wheel_fr: geometry collision cylinder length=0.10 radius=0.16; visual cylinder length=0.08 radius=0.09
- link wheel_rl: geometry collision cylinder length=0.10 radius=0.16; visual cylinder length=0.08 radius=0.09
- link wheel_rr: geometry collision cylinder length=0.10 radius=0.16; visual cylinder length=0.08 radius=0.09

Commit message: **

File: 200_html/urdf/vehicle/vehicle.urdf (robot description, URDF)
Before this commit: robot vehicle_4wd, 6 links, 5 joints
Links:
- link wheel_fl: geometry collision cylinder length=0.10 radius=0.16; visual cylinder length=0.06 radius=0.075
- link wheel_fr: geometry collision cylinder length=0.10 radius=0.16; visual cylinder length=0.06 radius=0.075
- link wheel_rl: geometry collision cylinder length=0.10 radius=0.16; visual cylinder length=0.06 radius=0.075
- link wheel_rr: geometry collision cylinder length=0.10 radius=0.16; visual cylinder length=0.06 radius=0.075

Commit message: **

File: 200_html/urdf/vehicle/vehicle.urdf (robot description, URDF)
Before this commit: robot vehicle_4wd, 6 links, 5 joints
Links:
- link wheel_fl: geometry collision cylinder length=0.10 radius=0.16; visual box size=0.010 0.145 0.024
- link wheel_fr: geometry collision cylinder length=0.10 radius=0.16; visual box size=0.010 0.145 0.024
- link wheel_rl: geometry collision cylinder length=0.10 radius=0.16; visual box size=0.010 0.145 0.024
- link wheel_rr: geometry collision cylinder length=0.10 radius=0.16; visual box size=0.010 0.145 0.024

Commit message: **

File: 200_html/urdf/vehicle/vehicle.urdf (robot description, URDF)
Before this commit: robot vehicle_4wd, 6 links, 5 joints
Links:
- link wheel_fl: geometry collision cylinder length=0.10 radius=0.16; visual box size=0.006 0.098 0.022
- link wheel_fr: geometry collision cylinder length=0.10 radius=0.16; visual box size=0.006 0.098 0.022
- link wheel_rl: geometry collision cylinder length=0.10 radius=0.16; visual box size=0.006 0.098 0.022
- link wheel_rr: geometry collision cylinder length=0.10 radius=0.16; visual box size=0.006 0.098 0.022

Commit message: **

File: 200_html/urdf/vehicle/vehicle.urdf (robot description, URDF)
Before this commit: robot vehicle_4wd, 6 links, 5 joints
Links:
- link wheel_fl: geometry collision cylinder length=0.10 radius=0.16; visual box size=0.010 0.098 0.028
- link wheel_fr: geometry collision cylinder length=0.10 radius=0.16; visual box size=0.010 0.098 0.028
- link wheel_rl: geometry collision cylinder length=0.10 radius=0.16; visual box size=0.010 0.098 0.028
- link wheel_rr: geometry collision cylinder length=0.10 radius=0.16; visual box size=0.010 0.098 0.028

Commit message: **

File: 200_html/urdf/vehicle/vehicle.urdf (robot description, URDF)
Before this commit: robot vehicle_4wd, 6 links, 5 joints
Links:
- link wheel_fl: geometry collision cylinder length=0.10 radius=0.16; visual box size=0.014 0.096 0.022
- link wheel_fr: geometry collision cylinder length=0.10 radius=0.16; visual box size=0.014 0.096 0.022
- link wheel_rl: geometry collision cylinder length=0.10 radius=0.16; visual box size=0.014 0.096 0.022
- link wheel_rr: geometry collision cylinder length=0.10 radius=0.16; visual box size=0.014 0.096 0.022

Commit message: **

File: 200_html/urdf/vehicle/vehicle.urdf (robot description, URDF)
Before this commit: robot vehicle_4wd, 6 links, 5 joints
Links:
- added link ground_patch; visual box size=2.00 1.80 0.005
Joints:
- added joint car_frame_to_ground_patch: type fixed, parent car_frame, child ground_patch, origin xyz=0.0566667 0 -0.1025 rpy=0 0 0

Commit message: 노면 길이 2배 증가

File: 200_html/urdf/vehicle/vehicle.urdf (robot description, URDF)
Before this commit: robot vehicle_4wd, 7 links, 6 joints
Links:
- link ground_patch: geometry visual box size=4.00 1.80 0.005

Commit message: ㅁㅁ

File: 200_html/urdf/vehicle/vehicle.urdf (robot description, URDF)
Before this commit: robot vehicle_4wd, 7 links, 6 joints
Links:
- link ground_patch: geometry visual box size=8.00 1.80 0.005

Commit message: ㅁㅁ

File: 200_html/urdf/vehicle/vehicle.urdf (robot description, URDF)
Before this commit: robot vehicle_4wd, 7 links, 6 joints
Links:
- link ground_patch: geometry visual box size=2.00 1.80 0.005

Commit message: aa

File: 200_html/urdf/vehicle/vehicle.urdf (robot description, URDF)
Before this commit: robot vehicle_4wd, 7 links, 6 joints
Links:
- added link ellipsoid_surface_patch; visual box size=2.42 2.3958 0.005
Joints:
- added joint base_to_ellipsoid_surface_patch: type fixed, parent base_link, child ellipsoid_surface_patch, origin xyz=0 0.0566667 -0.0025 rpy=0 0 0

Commit message: ㅁㅁ

File: 200_html/urdf/vehicle/vehicle.urdf (robot description, URDF)
Before this commit: robot vehicle_4wd, 8 links, 7 joints
Joints:
- joint base_to_ellipsoid_surface_patch: origin xyz=0 0.0566667 -0.0025 rpy=0 0 0 -> xyz=0 0.0566667 -0.3000 rpy=0 0 0

Commit message: ㅁㅁ

File: 200_html/urdf/vehicle/vehicle.urdf (robot description, URDF)
Before this commit: robot vehicle_4wd, 8 links, 7 joints
Links:
- link ellipsoid_surface_patch: geometry visual box size=4.84 4.7916 0.005

Commit message: aa

File: 200_html/urdf/vehicle/vehicle.urdf (robot description, URDF)
Before this commit: robot vehicle_4wd, 8 links, 7 joints
Links:
- removed link ellipsoid_surface_patch
- removed link ground_patch
- added link ellipsoid_surface; visual box size=4.84 4.7916 0.005
- added link ground; visual box size=2.00 1.80 0.005
Joints:
- removed joint base_to_car_frame
- removed joint base_to_ellipsoid_surface_patch
- removed joint car_frame_to_ground_patch
- added joint base_to_ellipsoid_surface: type fixed, parent base_link, child ellipsoid_surface, origin xyz=0 0.0566667 -0.3000 rpy=0 0 0
- added joint ellipsoid_surface_to_ground: type fixed, parent ellipsoid_surface, child ground, origin xyz=0 0 0.2975 rpy=0 0 1.5707963
- added joint ground_to_car_frame: type fixed, parent ground, child car_frame, origin xyz=-0.0566667 0 0.1025 rpy=0 0 0

Commit message: ㅁㅁ

File: 200_html/urdf/vehicle/vehicle.urdf (robot description, URDF)
Before this commit: robot vehicle_4wd, 8 links, 7 joints
Joints:
- joint ellipsoid_surface_to_ground: origin xyz=0 0 0.2975 rpy=0 0 1.5707963 -> xyz=0 0 0.2975 rpy=0 0 0

Commit message: aa

File: 200_html/urdf/vehicle/vehicle.urdf (robot description, URDF)
Before this commit: robot vehicle_4wd, 8 links, 7 joints
Links:
- link ground: geometry visual box size=2.00 1.80 0.005; visual sphere radius=0.05

Commit message: ㅁㅁ

File: 200_html/urdf/vehicle/vehicle.urdf (robot description, URDF)
Before this commit: robot vehicle_4wd, 8 links, 7 joints
Links:
- link ground: geometry visual box size=2.00 1.80 0.005; visual sphere radius=0.01

Commit message: ㅁㅁ

File: 200_html/urdf/vehicle/vehicle.urdf (robot description, URDF)
Before this commit: robot vehicle_4wd, 8 links, 7 joints
Links:
- link ground: geometry visual box size=2.00 1.80 0.005; visual sphere radius=0.015

Commit message: ㅁㅁ

File: 200_html/urdf/vehicle/vehicle.urdf (robot description, URDF)
Before this commit: robot vehicle_4wd, 8 links, 7 joints
Links:
- link ground: geometry visual box size=2.00 1.80 0.005; visual sphere radius=0.04

Commit message: ㅁㅁ

File: 200_html/urdf/vehicle/vehicle.urdf (robot description, URDF)
Before this commit: robot vehicle_4wd, 8 links, 7 joints
Joints:
- joint ellipsoid_surface_to_ground: origin xyz=0 0 0.2975 rpy=0 0 0 -> xyz=0 0 0.3000 rpy=0 0 0

Commit message: ㅁㅁ

File: 200_html/urdf/vehicle/vehicle.urdf (robot description, URDF)
Before this commit: robot vehicle_4wd, 8 links, 7 joints
Links:
- link base_link: geometry visual sphere radius=0.04
- link ground: geometry visual box size=2.00 1.80 0.005

Commit message: ㅁㅁ

File: 200_html/urdf/vehicle/vehicle.urdf (robot description, URDF)
Before this commit: robot vehicle_4wd, 8 links, 7 joints
Joints:
- joint base_to_ellipsoid_surface: origin xyz=0 0.0566667 -0.3000 rpy=0 0 0 -> xyz=0 0 -0.3000 rpy=0 0 0
- joint ground_to_car_frame: origin xyz=-0.0566667 0 0.1025 rpy=0 0 0 -> xyz=0 0 0.1025 rpy=0 0 0

Commit message: ㅁㅁ

File: 200_html/urdf/vehicle/vehicle.urdf (robot description, URDF)
Before this commit: robot vehicle_4wd, 8 links, 7 joints
Links:
- added link gear_fl, mass 0.12; visual cylinder length=0.065 radius=0.055
- added link gear_fr, mass 0.12; visual cylinder length=0.065 radius=0.055
- added link gear_rl, mass 0.12; visual cylinder length=0.065 radius=0.055
- added link gear_rr, mass 0.12; visual cylinder length=0.065 radius=0.055
Joints:
- added joint joint_gear_fl: type fixed, parent wheel_fl, child gear_fl, origin xyz=0 0 0 rpy=0 0 0
- added joint joint_gear_fr: type fixed, parent wheel_fr, child gear_fr, origin xyz=0 0 0 rpy=0 0 0
- added joint joint_gear_rl: type fixed, parent wheel_rl, child gear_rl, origin xyz=0 0 0 rpy=0 0 0
- added joint joint_gear_rr: type fixed, parent wheel_rr, child gear_rr, origin xyz=0 0 0 rpy=0 0 0

Commit message: ㅁㅁ

File: 200_html/urdf/vehicle/vehicle.urdf (robot description, URDF)
Before this commit: robot vehicle_4wd, 12 links, 11 joints
Links:
- added link obstacle_rock_01; collision sphere radius=0.14; visual sphere radius=0.14
Joints:
- added joint obstacle_rock_01_joint: type fixed, parent ground, child obstacle_rock_01, origin xyz=1.10 0.00 0.14 rpy=0 0 0

Commit message: ㅁㅁ

File: 200_html/urdf/vehicle/vehicle.urdf (robot description, URDF)
Before this commit: robot vehicle_4wd, 13 links, 12 joints
Links:
- link obstacle_rock_01: geometry collision box size=0.24 0.34 0.06; collision box size=0.44 0.34 0.08
Joints:
- joint obstacle_rock_01_joint: origin xyz=1.10 0.00 0.14 rpy=0 0 0 -> xyz=1.10 0.00 0.00 rpy=0 0 0

Commit message: ㅁㅁ

File: 200_html/urdf/vehicle/vehicle.urdf (robot description, URDF)
Before this commit: robot vehicle_4wd, 13 links, 12 joints
Links:
- link obstacle_rock_01: geometry collision box size=0.44 0.34 0.08; visual box size=0.44 0.34 0.08

Commit message: ㅁㅁ

File: 200_html/urdf/vehicle/vehicle.urdf (robot description, URDF)
Before this commit: robot vehicle_4wd, 13 links, 12 joints
Links:
- added link obstacle_rock_02; collision box size=0.44 0.60 0.08; visual box size=0.44 1.20 0.08
- link ground: geometry visual box size=4.00 2.80 0.005
- link obstacle_rock_01: geometry collision box size=0.44 0.34 0.08; visual box size=0.24 0.34 0.08
Joints:
- added joint obstacle_rock_02_joint: type fixed, parent ground, child obstacle_rock_02, origin xyz=1.48 0.0 0.00 rpy=0 0 0
- joint obstacle_rock_01_joint: origin xyz=1.10 0.00 0.00 rpy=0 0 0 -> xyz=0.88 0.40 0.00 rpy=0 0 0
