Commit message: ss

File: 200_html/urdf/sw_01/ASSY.urdf (robot description, URDF)
Before this commit: robot ASSY, 10 links, 9 joints
Links:
- link base_link: geometry collision mesh filename=../meshes/base_link.STL; visual mesh filename=../meshes/base_link.STL
- link front_left_pinion_link: geometry collision mesh filename=../meshes/front_left_pinion_link.STL; visual mesh filename=../meshes/front_left_pinion_link.STL
- link front_left_wheel_link: geometry collision mesh filename=../meshes/front_left_wheel_link.STL; visual mesh filename=../meshes/front_left_wheel_link.STL
- link front_right_pinion_link: geometry collision mesh filename=../meshes/front_right_pinion_link.STL; visual mesh filename=../meshes/front_right_pinion_link.STL
- link front_right_wheel_link: geometry collision mesh filename=../meshes/front_right_wheel_link.STL; visual mesh filename=../meshes/front_right_wheel_link.STL
- link rear_left_pinion_link: geometry collision mesh filename=../meshes/rear_left_pinion_link.STL; visual mesh filename=../meshes/rear_left_pinion_link.STL
- link rear_left_wheel_link: geometry collision mesh filename=../meshes/rear_left_wheel_link.STL; visual mesh filename=../meshes/rear_left_wheel_link.STL
- link rear_right_pinion_link: geometry collision mesh filename=../meshes/rear_right_pinion_link.STL; visual mesh filename=../meshes/rear_right_pinion_link.STL
- link rear_right_wheel_link: geometry collision mesh filename=../meshes/rear_right_wheel_link.STL; visual mesh filename=../meshes/rear_right_wheel_link.STL
- link swing_Link: geometry collision mesh filename=../meshes/swing_Link.STL; visual mesh filename=../meshes/swing_Link.STL

Commit message: aa

File: 200_html/urdf/sw_01/ASSY.urdf (robot description, URDF)
Before this commit: robot ASSY, 10 links, 9 joints
Links:
- link base_link: geometry collision mesh filename=./meshes/base_link.STL; visual mesh filename=./meshes/base_link.STL
- link front_left_pinion_link: geometry collision mesh filename=./meshes/front_left_pinion_link.STL; visual mesh filename=./meshes/front_left_pinion_link.STL
- link front_left_wheel_link: geometry collision mesh filename=./meshes/front_left_wheel_link.STL; visual mesh filename=./meshes/front_left_wheel_link.STL
- link front_right_pinion_link: geometry collision mesh filename=./meshes/front_right_pinion_link.STL; visual mesh filename=./meshes/front_right_pinion_link.STL
- link front_right_wheel_link: geometry collision mesh filename=./meshes/front_right_wheel_link.STL; visual mesh filename=./meshes/front_right_wheel_link.STL
- link rear_left_pinion_link: geometry collision mesh filename=./meshes/rear_left_pinion_link.STL; visual mesh filename=./meshes/rear_left_pinion_link.STL
- link rear_left_wheel_link: geometry collision mesh filename=./meshes/rear_left_wheel_link.STL; visual mesh filename=./meshes/rear_left_wheel_link.STL
- link rear_right_pinion_link: geometry collision mesh filename=./meshes/rear_right_pinion_link.STL; visual mesh filename=./meshes/rear_right_pinion_link.STL
- link rear_right_wheel_link: geometry collision mesh filename=./meshes/rear_right_wheel_link.STL; visual mesh filename=./meshes/rear_right_wheel_link.STL
- link swing_Link: geometry collision mesh filename=./meshes/swing_Link.STL; visual mesh filename=./meshes/swing_Link.STL
