Commit message: aa

File: 200_html/urdf/sw_02/urdf/ASSY.urdf (robot description, URDF)
Before this commit: robot ASSY, 12 links, 11 joints
Links:
- link base_link: geometry collision mesh filename=../meshes/meshes/base_link.STL; visual mesh filename=../meshes/meshes/base_link.STL
- link pinion_fl: geometry collision mesh filename=../meshes/meshes/front_left_pinion_link.STL; visual mesh filename=../meshes/meshes/front_left_pinion_link.STL
- link pinion_fr: geometry collision mesh filename=../meshes/meshes/front_right_pinion_link.STL; visual mesh filename=../meshes/meshes/front_right_pinion_link.STL
- link pinion_rl: geometry collision mesh filename=../meshes/meshes/rear_left_pinion_link.STL; visual mesh filename=../meshes/meshes/rear_left_pinion_link.STL
- link pinion_rr: geometry collision mesh filename=../meshes/meshes/rear_right_pinion_link.STL; visual mesh filename=../meshes/meshes/rear_right_pinion_link.STL
- link swing_link: geometry collision mesh filename=../meshes/meshes/swing_Link.STL; visual mesh filename=../meshes/meshes/swing_Link.STL
- link wheel_fl: geometry collision mesh filename=../meshes/meshes/front_left_wheel_link.STL; visual mesh filename=../meshes/meshes/front_left_wheel_link.STL
- link wheel_fr: geometry collision mesh filename=../meshes/meshes/front_right_wheel_link.STL; visual mesh filename=../meshes/meshes/front_right_wheel_link.STL
- link wheel_rl: geometry collision mesh filename=../meshes/meshes/rear_left_wheel_link.STL; visual mesh filename=../meshes/meshes/rear_left_wheel_link.STL
- link wheel_rr: geometry collision mesh filename=../meshes/meshes/rear_right_wheel_link.STL; visual mesh filename=../meshes/meshes/rear_right_wheel_link.STL

Commit message: aa

File: 200_html/urdf/sw_02/urdf/ASSY.urdf (robot description, URDF)
Before this commit: robot ASSY, 12 links, 11 joints
Links:
- link base_link: geometry collision mesh filename=../meshes/base_link.STL; visual mesh filename=../meshes/base_link.STL
- link pinion_fl: geometry collision mesh filename=../meshes/front_left_pinion_link.STL; visual mesh filename=../meshes/front_left_pinion_link.STL
- link pinion_fr: geometry collision mesh filename=../meshes/front_right_pinion_link.STL; visual mesh filename=../meshes/front_right_pinion_link.STL
- link pinion_rl: geometry collision mesh filename=../meshes/rear_left_pinion_link.STL; visual mesh filename=../meshes/rear_left_pinion_link.STL
- link pinion_rr: geometry collision mesh filename=../meshes/rear_right_pinion_link.STL; visual mesh filename=../meshes/rear_right_pinion_link.STL
- link swing_link: geometry collision mesh filename=../meshes/swing_Link.STL; visual mesh filename=../meshes/swing_Link.STL
- link wheel_fl: geometry collision mesh filename=../meshes/front_left_wheel_link.STL; visual mesh filename=../meshes/front_left_wheel_link.STL
- link wheel_fr: geometry collision mesh filename=../meshes/front_right_wheel_link.STL; visual mesh filename=../meshes/front_right_wheel_link.STL
- link wheel_rl: geometry collision mesh filename=../meshes/rear_left_wheel_link.STL; visual mesh filename=../meshes/rear_left_wheel_link.STL
- link wheel_rr: geometry collision mesh filename=../meshes/rear_right_wheel_link.STL; visual mesh filename=../meshes/rear_right_wheel_link.STL
