Commit message: aa

File: 200_html/urdf/sw_05/urdf/ASSY.urdf (robot description, URDF)
Before this commit: robot 0724_urdf, 20 links, 19 joints
Links:
- link car_frame: geometry collision mesh filename=../meshes/car_frame.STL; visual mesh filename=../meshes/car_frame.STL
- link swing_link: geometry collision mesh filename=../meshes/swing_link.STL; visual mesh filename=../meshes/swing_link.STL
- link tire_fl: geometry collision mesh filename=../meshes/tire_fl.STL; visual mesh filename=../meshes/tire_fl.STL
- link tire_fr: geometry collision mesh filename=../meshes/tire_fr.STL; visual mesh filename=../meshes/tire_fr.STL
- link tire_rl: geometry collision mesh filename=../meshes/tire_rl.STL; visual mesh filename=../meshes/tire_rl.STL
- link tire_rr: geometry collision mesh filename=../meshes/tire_rr.STL; visual mesh filename=../meshes/tire_rr.STL
- link wheel_fl: geometry collision mesh filename=../meshes/wheel_fl.STL; visual mesh filename=../meshes/wheel_fl.STL
- link wheel_fr: geometry collision mesh filename=../meshes/wheel_fr.STL; visual mesh filename=../meshes/wheel_fr.STL
- link wheel_rl: geometry collision mesh filename=../meshes/wheel_rl.STL; visual mesh filename=../meshes/wheel_rl.STL
- link wheel_rr: geometry collision mesh filename=../meshes/wheel_rr.STL; visual mesh filename=../meshes/wheel_rr.STL
