Commit message: ㅁㅁ

File: 200_html/urdf/model/vehicle/vehicle.urdf (robot description, URDF)
Before this commit: robot vehicle_4wd, 14 links, 13 joints
Links:
- removed link base_link
- added link origin, mass 0.001; visual sphere radius=0.04
Joints:
- removed joint base_to_ellipsoid_surface
- removed joint ellipsoid_surface_to_ground
- added joint ground_to_ellipsoid_surface: type fixed, parent ground, child ellipsoid_surface, origin xyz=0 0 -0.3000 rpy=0 0 0
- added joint origin_to_ground: type fixed, parent origin, child ground, origin xyz=0 0 0 rpy=0 0 0

Commit message: ㅁㅁ

File: 200_html/urdf/model/vehicle/vehicle.urdf (robot description, URDF)
Before this commit: robot vehicle_4wd, 14 links, 13 joints
Links:
- link origin: mass 0.001 -> None

Commit message: ㅁㅁ

File: 200_html/urdf/model/vehicle/vehicle.urdf (robot description, URDF)
Before this commit: robot vehicle_4wd, 14 links, 13 joints
Links:
- link ellipsoid_surface: geometry visual box size=9.68 4.7916 0.005
- link ground: geometry visual box size=8.00 2.80 0.005
Joints:
- joint obstacle_rock_02_joint: origin xyz=1.48 0.0 0.00 rpy=0 0 0 -> xyz=1.68 0.0 0.00 rpy=0 0 0

Commit message: ㅁㅁ

File: 200_html/urdf/model/vehicle/vehicle.urdf (robot description, URDF)
Before this commit: robot vehicle_4wd, 14 links, 13 joints
Links:
- added link obstacle_rock_03; collision box size=0.44 0.60 0.08; visual box size=0.44 1.20 0.08
- link obstacle_rock_02: geometry collision box size=0.44 0.34 0.08; visual box size=0.24 0.34 0.08
Joints:
- added joint obstacle_rock_03_joint: type fixed, parent ground, child obstacle_rock_03, origin xyz=2.88 0.0 0.00 rpy=0 0 0
- joint obstacle_rock_01_joint: origin xyz=0.88 0.40 0.00 rpy=0 0 0 -> xyz=0.88 0.00 0.00 rpy=0 0 0
- joint obstacle_rock_02_joint: origin xyz=1.68 0.0 0.00 rpy=0 0 0 -> xyz=1.88 0.40 0.00 rpy=0 0 0

Commit message: aa

File: 200_html/urdf/model/vehicle/vehicle.urdf (robot description, URDF)
Before this commit: robot vehicle_4wd, 15 links, 14 joints
Links:
- link obstacle_rock_01: geometry collision box size=0.44 0.34 0.05; visual box size=0.24 0.34 0.05
- link obstacle_rock_02: geometry collision box size=0.44 0.34 0.05; visual box size=0.24 0.34 0.05
- link obstacle_rock_03: geometry collision box size=0.44 0.60 0.05; visual box size=0.44 1.20 0.05

Commit message: ㅁㅁ

File: 200_html/urdf/model/vehicle/vehicle.urdf (robot description, URDF)
Before this commit: robot vehicle_4wd, 15 links, 14 joints
Links:
- added link hole_01; visual box size=0.44 0.34 0.05
- link ellipsoid_surface: geometry visual box size=12.584 4.7916 0.005
- link ground: geometry visual box size=10.40 2.80 0.005
- link obstacle_rock_02: geometry collision box size=0.44 0.60 0.05; visual box size=0.44 1.20 0.05
- link obstacle_rock_03: geometry collision box size=0.44 0.34 0.05; visual box size=0.24 0.34 0.05
Joints:
- added joint hole_01_joint: type fixed, parent ground, child hole_01, origin xyz=3.88 0.40 0.00 rpy=0 0 0
- joint obstacle_rock_02_joint: origin xyz=1.88 0.40 0.00 rpy=0 0 0 -> xyz=1.88 0.0 0.00 rpy=0 0 0
- joint obstacle_rock_03_joint: origin xyz=2.88 0.0 0.00 rpy=0 0 0 -> xyz=2.88 0.40 0.00 rpy=0 0 0

Commit message: ㅁㅁ

File: 200_html/urdf/model/vehicle/vehicle.urdf (robot description, URDF)
Before this commit: robot vehicle_4wd, 16 links, 15 joints
Links:
- link ground: geometry visual box size=10.40 2.80 0.50
Joints:
- joint ground_to_ellipsoid_surface: origin xyz=0 0 -0.3000 rpy=0 0 0 -> xyz=0 0 -0.5005 rpy=0 0 0

Commit message: ㅁㅁ

File: 200_html/urdf/model/vehicle/vehicle.urdf (robot description, URDF)
Before this commit: robot vehicle_4wd, 16 links, 15 joints
Links:
- link hole_01: geometry visual box size=0.16 0.34 0.05

Commit message: ㅁ

File: 200_html/urdf/model/vehicle/vehicle.urdf (robot description, URDF)
Before this commit: robot vehicle_4wd, 16 links, 15 joints
Links:
- link hole_01: geometry visual box size=0.32 1.20 0.05
Joints:
- joint hole_01_joint: origin xyz=3.88 0.40 0.00 rpy=0 0 0 -> xyz=3.88 0.00 0.00 rpy=0 0 0

Commit message: ㅁㅁ

File: 200_html/urdf/model/vehicle/vehicle.urdf (robot description, URDF)
Before this commit: robot vehicle_4wd, 16 links, 15 joints
Joints:
- joint ground_to_car_frame: origin xyz=0 0 0.1025 rpy=0 0 0 -> xyz=0 0 0.10 rpy=0 0 0

Commit message: ㅁㅁ

File: 200_html/urdf/model/vehicle/vehicle.urdf (robot description, URDF)
Before this commit: robot vehicle_4wd, 16 links, 15 joints
Links:
- link ground: geometry collision box size=10.40 2.80 0.50; visual box size=10.40 2.80 0.50

Commit message: ㅁㅁ

File: 200_html/urdf/model/vehicle/vehicle.urdf (robot description, URDF)
Before this commit: robot vehicle_4wd, 16 links, 15 joints
Joints:
- removed joint ground_to_ellipsoid_surface
- added joint origin_to_ellipsoid_surface: type fixed, parent origin, child ellipsoid_surface, origin xyz=0 0 -0.5005 rpy=0 0 0

Commit message: ㅁㅁ

File: 200_html/urdf/model/vehicle/vehicle.urdf (robot description, URDF)
Before this commit: robot vehicle_4wd, 16 links, 15 joints
Links:
- link ellipsoid_surface: geometry visual box size=15.1008 4.7916 0.005
- link ground: geometry collision box size=12.48 2.80 0.50; visual box size=12.48 2.80 0.50
Joints:
- joint hole_01_joint: origin xyz=3.88 0.00 0.00 rpy=0 0 0 -> xyz=5.42 0.00 0.00 rpy=0 0 0
- joint obstacle_rock_01_joint: origin xyz=0.88 0.00 0.00 rpy=0 0 0 -> xyz=1.39 0.00 0.00 rpy=0 0 0
- joint obstacle_rock_02_joint: origin xyz=1.88 0.0 0.00 rpy=0 0 0 -> xyz=2.7333 0.0 0.00 rpy=0 0 0
- joint obstacle_rock_03_joint: origin xyz=2.88 0.40 0.00 rpy=0 0 0 -> xyz=4.0767 0.00 0.00 rpy=0 0 0

Commit message: ㅁㅁ

File: 200_html/urdf/model/vehicle/vehicle.urdf (robot description, URDF)
Before this commit: robot vehicle_4wd, 16 links, 15 joints
Joints:
- joint obstacle_rock_03_joint: origin xyz=4.0767 0.00 0.00 rpy=0 0 0 -> xyz=4.0767 0.40 0.00 rpy=0 0 0

Commit message: ㅁㅁ

File: 200_html/urdf/model/vehicle/vehicle.urdf (robot description, URDF)
Before this commit: robot vehicle_4wd, 16 links, 15 joints
Links:
- link obstacle_rock_03: geometry collision box size=0.44 0.34 0.025; visual box size=0.24 0.34 0.025

Commit message: ㅁㅁ

File: 200_html/urdf/model/vehicle/vehicle.urdf (robot description, URDF)
Before this commit: robot vehicle_4wd, 16 links, 15 joints
Links:
- link gear_fl: geometry visual box size=0.010 0.018 0.008; visual box size=0.010 0.018 0.008
- link gear_fr: geometry visual box size=0.010 0.018 0.008; visual box size=0.010 0.018 0.008
- link gear_rl: geometry visual box size=0.010 0.018 0.008; visual box size=0.010 0.018 0.008
- link gear_rr: geometry visual box size=0.010 0.018 0.008; visual box size=0.010 0.018 0.008

Commit message: ㅁㅁ

File: 200_html/urdf/model/vehicle/vehicle.urdf (robot description, URDF)
Before this commit: robot vehicle_4wd, 16 links, 15 joints
Links:
- link gear_fl: geometry visual box size=0.010 0.024 0.009; visual box size=0.010 0.024 0.009
- link gear_fr: geometry visual box size=0.010 0.024 0.009; visual box size=0.010 0.024 0.009
- link gear_rl: geometry visual box size=0.010 0.024 0.009; visual box size=0.010 0.024 0.009
- link gear_rr: geometry visual box size=0.010 0.024 0.009; visual box size=0.010 0.024 0.009
Joints:
- joint joint_gear_fl: origin xyz=0.33 0.40 0.06 rpy=0 0 0 -> xyz=0.33 0.47 0.06 rpy=0 0 0
- joint joint_gear_fr: origin xyz=0.33 -0.40 0.06 rpy=0 0 0 -> xyz=0.33 -0.47 0.06 rpy=0 0 0
- joint joint_gear_rl: origin xyz=-0.33 0.40 0.06 rpy=0 0 0 -> xyz=-0.33 0.47 0.06 rpy=0 0 0
- joint joint_gear_rr: origin xyz=-0.33 -0.40 0.06 rpy=0 0 0 -> xyz=-0.33 -0.47 0.06 rpy=0 0 0
