Commit message: aa

File: 200_html/urdf/model/sw_08/urdf/sw.urdf (robot description, URDF)
Before this commit: robot sw9, 20 links, 19 joints
Links:
- removed link base_link
- added link car_frame, mass 4.36726752622486; collision mesh filename=../meshes/base_link.STL; visual mesh filename=../meshes/base_link.STL
Joints:
- removed joint ground_to_base_link_joint
- added joint ground_to_car_frame_joint: type fixed, parent ground, child car_frame, origin xyz=0 0 0.005 rpy=0 0 0
- joint ground_to_hemisphere_joint: origin xyz=0.0 -1.0 0.005 rpy=0 0 0 -> xyz=1.55 0.0 0.005 rpy=0 0 0
- joint inner_gear_rl_joint: parent base_link -> car_frame
- joint inner_gear_rr_joint: parent base_link -> car_frame
- joint inner_wheel_rl_joint: parent base_link -> car_frame
- joint inner_wheel_rr_joint: parent base_link -> car_frame
- joint swing_joint: parent base_link -> car_frame

Commit message: aa

File: 200_html/urdf/model/sw_08/urdf/sw.urdf (robot description, URDF)
Before this commit: robot sw9, 20 links, 19 joints
Links:
- link obstacle_rock_1: geometry collision box size=0.14 0.16 0.07; visual box size=0.14 0.16 0.03

Commit message: aa

File: 200_html/urdf/model/sw_08/urdf/sw.urdf (robot description, URDF)
Before this commit: robot sw9, 20 links, 19 joints
Links:
- link obstacle_rock_1: geometry collision box size=0.14 0.16 0.07; visual box size=0.14 0.16 0.01

Commit message: ㅁㅁ

File: 200_html/urdf/model/sw_08/urdf/sw.urdf (robot description, URDF)
Before this commit: robot sw9, 20 links, 19 joints
Links:
- link obstacle_rock_1: geometry collision box size=0.14 0.16 0.01; visual box size=0.14 0.16 0.01
Joints:
- joint ground_to_rock_1_joint: origin xyz=0.7 0.3 0.04 rpy=0 0 0 -> xyz=0.7 0.3 0.005 rpy=0 0 0

Commit message: ㅁㅁ

File: 200_html/urdf/model/sw_08/urdf/sw.urdf (robot description, URDF)
Before this commit: robot sw9, 20 links, 19 joints
Links:
- link obstacle_rock_1: geometry collision box size=0.14 0.16 0.05; visual box size=0.14 0.16 0.05
Joints:
- joint ground_to_rock_1_joint: origin xyz=0.7 0.3 0.005 rpy=0 0 0 -> xyz=0.7 0.3 0.025 rpy=0 0 0

Commit message: ㅁㅁ

File: 200_html/urdf/model/sw_08/urdf/sw.urdf (robot description, URDF)
Before this commit: robot sw9, 20 links, 19 joints
Links:
- link obstacle_rock_1: geometry collision box size=0.14 0.16 0.01; visual box size=0.14 0.16 0.01
Joints:
- joint ground_to_rock_1_joint: origin xyz=0.7 0.3 0.025 rpy=0 0 0 -> xyz=0.7 0.3 0.01 rpy=0 0 0
