Commit message: ㅁㅁ

File: 200_html/urdf/model/sw_10/urdf/sw.urdf (robot description, URDF)
Before this commit: robot sw5, 30 links, 29 joints
Links:
- link version_marker: geometry collision mesh filename=../meshes/version_marker.STL scale=0.01 0.01 0.01; visual mesh filename=../meshes/version_marker.STL scale=0.01 0.01 0.01
