Commit message: ㅁㅁ

File: 200_html/urdf/model/sw_13/urdf/sw.urdf (robot description, URDF)
Before this commit: robot sw5, 30 links, 29 joints
Joints:
- joint ground_to_rock_1_joint: origin xyz=1.801 0.315 0.04 rpy=0 0 0 -> xyz=-1.801 0.315 0.04 rpy=0 0 0
- joint ground_to_wood_bar_joint: origin xyz=3.730 0.0 0.035 rpy=0 0 0 -> xyz=-3.730 0.0 0.035 rpy=0 0 0

Commit message: ㅁㅁ

File: 200_html/urdf/model/sw_13/urdf/sw.urdf (robot description, URDF)
Before this commit: robot sw5, 30 links, 29 joints
Joints:
- joint ground_to_rock_1_joint: origin xyz=-1.801 0.315 0.04 rpy=0 0 0 -> xyz=1.801 0.315 0.04 rpy=0 0 0
- joint ground_to_wood_bar_joint: origin xyz=-3.730 0.0 0.035 rpy=0 0 0 -> xyz=3.730 0.0 0.035 rpy=0 0 0
