Commit message: ㅁㅁ

File: 200_html/urdf/model/sw_14/urdf/sw.urdf (robot description, URDF)
Before this commit: robot sw5, 30 links, 29 joints
Joints:
- joint ground_to_pothole_joint: origin xyz=0.0 -2.573 0.005 rpy=0 0 0 -> xyz=3.6 0.32225 0.005 rpy=0 0 0
- joint ground_to_rock_1_joint: origin xyz=1.801 0.315 0.04 rpy=0 0 0 -> xyz=2.4 0.32225 0.04 rpy=0 0 0
- joint ground_to_wood_bar_joint: origin xyz=3.730 0.0 0.035 rpy=0 0 0 -> xyz=1.2 0 0.035 rpy=0 0 0

Commit message: ㅁㅁ

File: 200_html/urdf/model/sw_14/urdf/sw.urdf (robot description, URDF)
Before this commit: robot sw5, 30 links, 29 joints
Links:
- link ground: geometry collision box size=8.786 6.5 0.2; visual box size=8.786 6.5 0.2
Joints:
- joint ellipsoid_to_ground_joint: origin xyz=0 0 0.30 rpy=0 0 0 -> xyz=0 0 0.20 rpy=0 0 0
- joint ground_to_car_frame_joint: origin xyz=0 0 0.0239 rpy=0 0 0 -> xyz=0 0 0.1189 rpy=0 0 0
- joint ground_to_pothole_joint: origin xyz=3.6 0.32225 0.005 rpy=0 0 0 -> xyz=3.6 0.32225 0.1 rpy=0 0 0
- joint ground_to_rock_1_joint: origin xyz=2.4 0.32225 0.04 rpy=0 0 0 -> xyz=2.4 0.32225 0.135 rpy=0 0 0
- joint ground_to_sphere_joint: origin xyz=0 0 0.0 rpy=0 0 0 -> xyz=0 0 0.095 rpy=0 0 0
- joint ground_to_wood_bar_joint: origin xyz=1.2 0 0.035 rpy=0 0 0 -> xyz=1.2 0 0.13 rpy=0 0 0

Commit message: ㅁㅁ

File: 200_html/urdf/model/sw_14/urdf/sw.urdf (robot description, URDF)
Before this commit: robot sw5, 30 links, 29 joints
Joints:
- joint ground_to_pothole_joint: origin xyz=3.6 0.32225 0.1 rpy=0 0 0 -> xyz=3.6 0.24 0.1 rpy=0 0 0
