Commit message: ㅁㅁ

File: 200_html/urdf/model/sw_16/urdf/sw.urdf (robot description, URDF)
Before this commit: robot sw5, 34 links, 33 joints
Links:
- link gear_marker_fl: geometry collision mesh filename=../meshes/gear_marker_fl.STL; visual mesh filename=../meshes/gear_marker_fl.STL
- link gear_marker_fr: geometry collision mesh filename=../meshes/gear_marker_fr.STL; visual mesh filename=../meshes/gear_marker_fr.STL
- link gear_marker_rl: geometry collision mesh filename=../meshes/gear_marker_rl.STL; visual mesh filename=../meshes/gear_marker_rl.STL
- link gear_marker_rr: geometry collision mesh filename=../meshes/gear_marker_rr.STL; visual mesh filename=../meshes/gear_marker_rr.STL
