Commit message: ㅁㅁ

File: 200_html/urdf/model/sw_17/urdf/sw17.urdf (robot description, URDF)
Before this commit: robot sw5, 34 links, 33 joints
Links:
- link car_frame: geometry collision mesh filename=package://sw17/meshes/car_frame.STL; visual mesh filename=package://sw17/meshes/car_frame.STL
- link cover_fl: geometry collision mesh filename=package://sw17/meshes/cover_fl.STL; visual mesh filename=package://sw17/meshes/cover_fl.STL
- link cover_fr: geometry collision mesh filename=package://sw17/meshes/cover_fr.STL; visual mesh filename=package://sw17/meshes/cover_fr.STL
- link cover_rl: geometry collision mesh filename=package://sw17/meshes/cover_rl.STL; visual mesh filename=package://sw17/meshes/cover_rl.STL
- link cover_rr: geometry collision mesh filename=package://sw17/meshes/cover_rr.STL; visual mesh filename=package://sw17/meshes/cover_rr.STL
- link gear_marker_fl: geometry collision mesh filename=package://sw17/meshes/gear_marker_fl.STL; visual mesh filename=package://sw17/meshes/gear_marker_fl.STL
- link gear_marker_fr: geometry collision mesh filename=package://sw17/meshes/gear_marker_fr.STL; visual mesh filename=package://sw17/meshes/gear_marker_fr.STL
- link gear_marker_rl: geometry collision mesh filename=package://sw17/meshes/gear_marker_rl.STL; visual mesh filename=package://sw17/meshes/gear_marker_rl.STL
- link gear_marker_rr: geometry collision mesh filename=package://sw17/meshes/gear_marker_rr.STL; visual mesh filename=package://sw17/meshes/gear_marker_rr.STL
- link inner_gear_fl: geometry collision mesh filename=package://sw17/meshes/inner_gear_fl.STL; visual mesh filename=package://sw17/meshes/inner_gear_fl.STL
- link inner_gear_fr: geometry collision mesh filename=package://sw17/meshes/inner_gear_fr.STL; visual mesh filename=package://sw17/meshes/inner_gear_fr.STL
- link inner_gear_rl: geometry collision mesh filename=package://sw17/meshes/inner_gear_rl.STL; visual mesh filename=package://sw17/meshes/inner_gear_rl.STL
- link inner_gear_rr: geometry collision mesh filename=package://sw17/meshes/inner_gear_rr.STL; visual mesh filename=package://sw17/meshes/inner_gear_rr.STL
- link inner_wheel_fl: geometry collision mesh filename=package://sw17/meshes/inner_wheel_fl.STL; visual mesh filename=package://sw17/meshes/inner_wheel_fl.STL
- link inner_wheel_fr: geometry collision mesh filename=package://sw17/meshes/inner_wheel_fr.STL; visual mesh filename=package://sw17/meshes/inner_wheel_fr.STL
- link inner_wheel_rl: geometry collision mesh filename=package://sw17/meshes/inner_wheel_rl.STL; visual mesh filename=package://sw17/meshes/inner_wheel_rl.STL
- link inner_wheel_rr: geometry collision mesh filename=package://sw17/meshes/inner_wheel_rr.STL; visual mesh filename=package://sw17/meshes/inner_wheel_rr.STL
- link marker_fl: geometry collision mesh filename=package://sw17/meshes/marker_fl.STL; visual mesh filename=package://sw17/meshes/marker_fl.STL
- link marker_fr: geometry collision mesh filename=package://sw17/meshes/marker_fr.STL; visual mesh filename=package://sw17/meshes/marker_fr.STL
- link marker_rl: geometry collision mesh filename=package://sw17/meshes/marker_rl.STL; visual mesh filename=package://sw17/meshes/marker_rl.STL
- link marker_rr: geometry collision mesh filename=package://sw17/meshes/marker_rr.STL; visual mesh filename=package://sw17/meshes/marker_rr.STL
- link obstacle_pothole: geometry collision mesh filename=package://sw17/meshes/pothole.STL scale=0.01 0.01 0.01; visual mesh filename=package://sw17/meshes/pothole.STL scale=0.01 0.01 0.01
- link obstacle_wood_bar: geometry collision box size=0.10 1.5 0.05; visual box size=0.10 1.5 0.05
- link swing_link: geometry collision mesh filename=package://sw17/meshes/swing_link.STL; visual mesh filename=package://sw17/meshes/swing_link.STL
- link version_marker: geometry collision mesh filename=package://sw17/meshes/version_marker.STL scale=0.01 0.01 0.01; visual mesh filename=package://sw17/meshes/version_marker.STL scale=0.01 0.01 0.01
- link wheel_fl: geometry collision mesh filename=package://sw17/meshes/wheel_fl.STL; visual mesh filename=package://sw17/meshes/wheel_fl.STL
- link wheel_fr: geometry collision mesh filename=package://sw17/meshes/wheel_fr.STL; visual mesh filename=package://sw17/meshes/wheel_fr.STL
- link wheel_rl: geometry collision mesh filename=package://sw17/meshes/wheel_rl.STL; visual mesh filename=package://sw17/meshes/wheel_rl.STL
- link wheel_rr: geometry collision mesh filename=package://sw17/meshes/wheel_rr.STL; visual mesh filename=package://sw17/meshes/wheel_rr.STL
Joints:
- removed joint inner_gear_rl_joint
- added joint inner_gaer_rl_joint: type continuous, parent swing_link, child inner_gear_rl, origin xyz=0 -0.133 0.32225 rpy=0 0 -0.059958, axis 0 0 1
- joint cover_fl_joint: origin xyz=-0.00287628069627605 0.0479137455158353 0.00774999999999976 rpy=3.14159265358979 0 -3.08163422030932 -> xyz=-0.0028763 0.047914 0.00775 rpy=3.1416 0 -3.0816
- joint gear_marker_fr_joint: origin xyz=0 0 0.006 rpy=0 0 0 -> xyz=0 0 0.00600000000000001 rpy=0 0 0
- joint gear_marker_rl_joint: origin xyz=0 0 0.00600000000000001 rpy=0 0 0 -> xyz=0 0 0.006 rpy=0 0 0
- joint gear_marker_rr_joint: origin xyz=0 0 0.00600000000000001 rpy=0 0 0 -> xyz=0 0 0.006 rpy=0 0 0

Commit message: ㅁㅁ

File: 200_html/urdf/model/sw_17/urdf/sw17.urdf (robot description, URDF)
Before this commit: robot sw5, 34 links, 33 joints
Joints:
- removed joint inner_gaer_rl_joint
- added joint inner_gear_rl_joint: type continuous, parent swing_link, child inner_gear_rl, origin xyz=0 -0.133 0.32225 rpy=0 0 -0.059958, axis 0 0 1
